File: mcmc12.brd (EAGLE design)
At the start: 48 x 40 mm, 60 parts, among them IC1 MCP73871, IC3 BGM123, IC4 CP2012N-20, IC5 TPS63001, J1 FTSH-105-01-L-DV-K, SW2 AYZ0102AGRLC, X2 USBi, Y1 12.28MHz

Commit message: Release v0.5.
Parts:
- added C27: 0.1uF, rcl:C1608
- added JP1, JP2, JP3, JP4: (no value), SparkFun:SJ_2S-NO
- added U$5: (no value), tkrworks:LOGO2
- C21, C23: value 47uF -> 220uF; device rcl:C2012 -> rcl:R/2012-12R
- R12, R13: value 49k9 -> 113k
- R23: device SparkFun:0603-RES -> SparkFun:0402-RES
- SV1: device con-lstb:MA06-2 -> pinhead:2X06
- SV2: device con-lstb:MA12-2 -> pinhead:2X12
- U$1: value MICRO_USB_HIROSE -> MICRO_USB_HIROSEZX-B; device tkrworks:MICRO_USB_HIROSE -> tkrworks:MICRO_USB_HIROSE_B
- moved U$1 2.70 mm to (43.5, 15.4)
- moved R12 1.00 mm to (28.2, 6.83)
- moved C23 0.96 mm to (29.7, 7.47), turned to 90 degrees
- moved R13 0.55 mm to (24.7, 6.83)
- moved C21 0.52 mm to (26.2, 7.47), turned to 90 degrees
- moved R14 0.35 mm to (21.6, 14.4)
- moved R15 0.30 mm to (20.5, 14.4)
Connections:
- new net N$10: JP4.1, R10.2
- new net N$6: JP1.1, R7.2
- new net N$7: JP2.1, R8.2
- new net N$8: JP3.1, R9.2
- net GND: now also C27.2; no longer SV2.14
- net HPOUTL: now also C21.+; no longer C21.1
- net HPOUTR: now also C23.+; no longer C23.1
- net MIC0: now also JP1.2; no longer R7.2
- net MIC1: now also JP2.2; no longer R8.2
- net MIC2: now also JP3.2; no longer R9.2
- net MIC3: now also JP4.2; no longer R10.2
- net OUTL: now also C21.-; no longer C21.2
- net OUTR: now also C23.-; no longer C23.2
- net SCL: now also SV2.14
- net SDA: now also SV2.13
- net VBUS: now also C27.1
- net VDD: no longer SV2.13
Routing:
- net N$10: track 0.00 -> 3.55 mm, vias 0 -> 1
- net N$7: track 0.00 -> 2.99 mm, vias 0 -> 1
- net N$8: track 0.00 -> 2.92 mm, vias 0 -> 1
- net VBUS: track 20.9 -> 23.7 mm
- net N$6: track 0.00 -> 2.69 mm, vias 0 -> 1
- net MIC0: track 7.38 -> 5.47 mm
- net SDA: track 66.2 -> 64.4 mm, vias 4 -> 3
- net MIC1: track 7.50 -> 5.80 mm
- net N$18: track 16.2 -> 14.5 mm
- net MIC3: track 8.04 -> 6.48 mm
- net MIC2: track 7.62 -> 6.14 mm
- net HPOUTL: track 20.2 -> 21.6 mm
- net D+: track 18.9 -> 17.6 mm
- net N$29: track 17.1 -> 16.2 mm
- net GND: track 133.1 -> 134.0 mm, vias 80 -> 81
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Other:
- board text added: "3V3 x2"
- board text added: "ADCSDATA1"
- board text added: "ADC_SDATA0"
- board text added: "BCLK"
- board text added: "DAC_SDATA"
- board text added: "GND x2"
- board text added: "GND x6"
- board text added: "IN0"
- board text added: "IN1"
- board text added: "IN2"
- board text added: "IN3"
- board text added: "LRCLK"
- board text added: "Li-Po"
- board text added: "MCLK"
- board text added: "MICBIAS"
- board text added: "OFF"
- board text added: "ON"
- board text added: "OUTL"
- board text added: "OUTR"
- board text added: "PA0"
- board text added: "PA1"
- board text added: "PA2"
- board text added: "PA3"
- board text added: "PA4"
- board text added: "PD10"
- board text added: "PD11"
- board text added: "PD12"
- board text added: "PD13"
- board text added: "PD14"
- board text added: "PD15"
- board text added: "PD9"
- board text added: "SCL"
- board text added: "SDA"
- board text added: "SWD"
- board text added: "USBi"
- board text added: "X"
- board text added: "Y"
- board text added: "Z"
- board text added: "v0.5"
- board text removed: "v0.3"

Commit message: Release v0.6.
Parts:
- C10, C13, C14, C15, C16, C18, C19, C20, C22, C24, C25, C26, C27: device rcl:C1608 -> rcl:C0402
- C21, C23: device rcl:R/2012-12R -> rcl:B/3528-21R
- moved C10 2.39 mm to (17.7, 27.6), turned to 180 degrees
- moved R13 2.25 mm to (26.9, 6.88)
- moved C15 1.60 mm to (18.4, 25.0), turned to 90 degrees
- moved C12 1.35 mm to (28.9, 28.3)
- moved C21 1.17 mm to (25.1, 7.88)
- moved C24 1.14 mm to (28.6, 13.0), turned to 0 degrees
- moved C17 1.03 mm to (17.7, 29.2), turned to 180 degrees
- moved C16 0.90 mm to (28.9, 26.6)
- moved C25 0.85 mm to (26.3, 11.4)
- moved C26 0.85 mm to (23.0, 11.4)
- moved U$3 0.53 mm to (24.9, 14.3)
- moved C23 0.43 mm to (29.9, 7.88)
- moved C18 0.43 mm to (17.6, 22.3)
- moved C27 0.35 mm to (31.4, 19.4)
- moved C11 0.35 mm to (19.2, 19.4)
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Connections:
- net GND: no longer U$3.25
Routing:
- net GND: track 134.0 -> 120.6 mm, vias 81 -> 71
- net VDD: track 59.7 -> 57.6 mm, vias 19 -> 18
- net CM: track 36.8 -> 34.9 mm
- net AIN0: track 19.8 -> 18.4 mm
- net MICBIAS0: track 26.1 -> 24.9 mm
- net HPOUTL: track 21.6 -> 20.5 mm
- net HPOUTR: track 24.1 -> 23.1 mm
- net VBUS: track 23.7 -> 24.5 mm
Other:
- board text added: "v0.6"
- board text removed: "v0.5"

Commit message: Release v0.7.
Parts:
- removed U$4: (no value), tkrworks:MIC
- removed U$5: (no value), tkrworks:LOGO2
- added JP5: (no value), SparkFun:1X02
- added LED2: (no value), led:CHIPLED_0603
- added R16, R17, R18, R19: 49k9, SparkFun:0402-RES
- added R20: 1k, SparkFun:0402-RES
- C21, C23: value 220uF -> 470uF
- R12, R13: value 113k -> 49k9
- SV1: device pinhead:2X06 -> pinhead-2:2X06ROUND
- moved R10 4.91 mm to (19.1, 15.5)
- moved R9 4.82 mm to (18.0, 15.5)
- moved R8 4.71 mm to (16.9, 15.5)
- moved R7 4.70 mm to (15.4, 15.5)
- moved R15 0.55 mm to (21.1, 14.4)
- moved R14 0.50 mm to (22.1, 14.4)
- moved C11 0.43 mm to (19.6, 19.3)
Connections:
- new net N$19: LED2.A, R20.1
- net GND: now also JP5.1, LED2.C, R16.2, R17.2, R18.2, R19.2
- net MIC0: now also R16.1
- net MIC1: now also R17.1
- net MIC2: now also R18.1
- net MIC3: now also R19.1
- net VBUS: now also JP5.2
- net VDD: now also R20.2
Routing:
- net GND: track 120.6 -> 138.1 mm, vias 71 -> 76
- net VBUS: track 24.5 -> 37.7 mm
- net N$14: track 0.00 -> 9.45 mm
- net N$13: track 0.00 -> 8.72 mm
- net N$12: track 0.00 -> 7.56 mm
- net N$16: track 0.00 -> 7.19 mm
- net MICBIAS0: track 24.9 -> 19.2 mm
- net N$8: track 2.92 -> 8.52 mm
- net MIC1: track 5.80 -> 11.1 mm, vias 0 -> 1
- net N$10: track 3.55 -> 8.50 mm
- net MIC3: track 6.48 -> 11.4 mm, vias 0 -> 1
- net MIC2: track 6.14 -> 11.0 mm, vias 0 -> 1
- net N$6: track 2.69 -> 7.37 mm
- net N$7: track 2.99 -> 7.67 mm
- net MIC0: track 5.47 -> 10.0 mm, vias 0 -> 1
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Other:
- board text added: "+5V"
- board text added: "GND"
- board text added: "MPU-9250"
- board text added: "uMI9s"
- board text added: "v0.7"
- board text removed: "MCMC12"
- board text removed: "v0.6"
