File: mcmc12.sch (EAGLE design)
At the start: 59 parts, among them IC1 MCP73871, IC3 BGM123, IC4 CP2012N-20, IC5 TPS63001, J1 FTSH-105-01-L-DV-K, SW2 AYZ0102AGRLC, X2 USBi, Y1 12.28MHz

Commit message: Release v0.5.
Parts:
- added C27: 0.1uF, rcl:C-EUC1608
- added JP1, JP2, JP3, JP4: (no value), SparkFun:JUMPER-2SMD-NO
- C21, C23: value 47uF -> 220uF; device rcl:C-EUC2012 -> rcl:CPOL-USR/2012-12R
- R12, R13: value 49k9 -> 113k
- R23: device SparkFun:RESISTOR0603-RES -> SparkFun:RESISTOR0402-RES
- SV1: device con-lstb:MA06-2 -> pinhead:PINHD-2X6
- SV2: device con-lstb:MA12-2 -> pinhead:PINHD-2X12
- U$1: value MICRO_USB_HIROSE -> MICRO_USB_HIROSEZX-B; device tkrworks:MICRO_USB_HIROSE -> tkrworks:MICRO_USB_HIROSEZX-B
Connections:
- new net N$10: JP4.1, R10.2
- new net N$6: JP1.1, R7.2
- new net N$7: JP2.1, R8.2
- new net N$8: JP3.1, R9.2
- net GND: now also C27.2; no longer SV2.14
- net HPOUTL: now also C21.+; no longer C21.1
- net HPOUTR: now also C23.+; no longer C23.1
- net MIC0: now also JP1.2; no longer R7.2
- net MIC1: now also JP2.2; no longer R8.2
- net MIC2: now also JP3.2; no longer R9.2
- net MIC3: now also JP4.2; no longer R10.2
- net OUTL: now also C21.-; no longer C21.2
- net OUTR: now also C23.-; no longer C23.2
- net SCL: now also SV2.14
- net SDA: now also SV2.13
- net VBUS: now also C27.1
- net VDD: no longer SV2.13
Other:
- moved on the sheet: C15, C24, C25, C26, R10, R14, R15, R7, R8, R9, U$3

Commit message: Release v0.6.
Parts:
- C10, C13, C14, C15, C16, C18, C19, C20, C22, C24, C25, C26, C27: device rcl:C-EUC1608 -> rcl:C-USC0402
- C21, C23: device rcl:CPOL-USR/2012-12R -> rcl:CPOL-USB/3528-21R
Connections:
- net GND: no longer U$3.PAD

Commit message: Release v0.7.
Parts:
- added JP5: (no value), SparkFun:M02PTH
- added LED2: (no value), led:LEDCHIPLED_0603
- added R16, R17, R18, R19: 49k9, SparkFun:RESISTOR0402-RES
- added R20: 1k, SparkFun:RESISTOR0402-RES
- C21, C23: value 220uF -> 470uF
- R12, R13: value 113k -> 49k9
- SV1: device pinhead:PINHD-2X6 -> pinhead-2:PINHD-2X06
Connections:
- new net N$19: LED2.A, R20.1
- net GND: now also JP5.1, LED2.C, R16.2, R17.2, R18.2, R19.2
- net MIC0: now also R16.1
- net MIC1: now also R17.1
- net MIC2: now also R18.1
- net MIC3: now also R19.1
- net VBUS: now also JP5.2
- net VDD: now also R20.2
Other:
- moved on the sheet: C15, JP1, JP2, JP3, JP4, R10, R7, R8, R9
