File: umi9s.brd (EAGLE design)
At the start: 48 x 40 mm, 71 parts, among them IC1 MCP73871, IC3 BGM123, IC4 CP2012N-20, IC5 TPS63001, J1 FTSH-105-01-L-DV-K, SW2 AYZ0102AGRLC, X2 USBi, Y1 12.28MHz

Commit message: Release v0.8.
Rename from mcmc12 to uMi9s.
Parts:
- SV2: device pinhead:2X12 -> pinhead-2:2X12ROUND
- moved C17 1.15 mm to (16.9, 28.4), turned to 90 degrees
- moved C10 1.10 mm to (18.4, 28.4), turned to 90 degrees
- moved C18 0.85 mm to (18.0, 21.6), turned to 270 degrees
- moved C27 0.45 mm to (30.9, 19.4)
- moved C13 0.05 mm to (21.1, 19.5)
Connections:
- net VBUS renamed N$14
Routing:
- net N$15: track 0.00 -> 17.2 mm
- net N$16: track 7.19 -> 22.3 mm
- net N$14 (its old number): track 9.45 -> 0.00 mm
- net GND: track 138.1 -> 144.7 mm, vias 76 -> 100
- net N$13: track 8.72 -> 4.43 mm
- net N$14: track 37.7 -> 40.5 mm, vias 6 -> 7
- net MICBIAS0: track 19.2 -> 17.0 mm, vias 4 -> 2
- net HPOUTR: track 23.1 -> 21.6 mm
- net D+: track 17.6 -> 19.1 mm
- net N$12: track 7.56 -> 8.96 mm
- net HPOUTL: track 20.5 -> 19.2 mm
- net D-: track 13.1 -> 14.2 mm
- net UART_CTS: track 20.5 -> 21.4 mm
- net CM: track 30.8 -> 31.4 mm
- net MCLKI: track 9.67 -> 9.02 mm
Other:
- board text added: "v0.8"
- board text removed: "v0.7"
