File: umi9s.sch (EAGLE design)
At the start: 71 parts, among them IC1 MCP73871, IC3 BGM123, IC4 CP2012N-20, IC5 TPS63001, J1 FTSH-105-01-L-DV-K, SW2 AYZ0102AGRLC, X2 USBi, Y1 12.28MHz

Commit message: Release v0.8.
Rename from mcmc12 to uMi9s.
Parts:
- SV2: device pinhead:PINHD-2X12 -> pinhead-2:PINHD-2X12
Connections:
- net VBUS renamed N$14
Changed lines of the file:
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@@
 <part name="VDD6" library="supply1" deviceset="VDD" device="" value="3V3"/>
 <part name="GND22" library="supply1" deviceset="GND" device=""/>
-<part name="U$1" library="tkrworks" library_urn="urn:adsk.eagle:library:1636359" deviceset="MICRO_USB_HIROSE" device="ZX-B" package3d_urn="urn:adsk.eagle:package:2471574/2" value="MICRO_USB_HIROSEZX-B"/>
+<part name="U$1" library="tkrworks" library_urn="urn:adsk.eagle:library:1636359" deviceset="MICRO_USB_HIROSE" device="ZX-B" package3d_urn="urn:adsk.eagle:package:2471574/3" value="MICRO_USB_HIROSEZX-B"/>
 <part name="IC3" library="tkrworks" library_urn="urn:adsk.eagle:library:1636359" deviceset="BGM12X" device="" package3d_urn="urn:adsk.eagle:package:1636513/2" value="BGM123"/>
 <part name="L1" library="rc-master-smd" deviceset="L_" device="1210" value="2.2uH"/>
@@
 <part name="VDD11" library="supply1" deviceset="VDD" device="" value="3V3"/>
 <part name="VDD12" library="supply1" deviceset="VDD" device="" value="3V3"/>
-<part name="SV2" library="pinhead" library_urn="urn:adsk.eagle:library:325" deviceset="PINHD-2X12" device="" package3d_urn="urn:adsk.eagle:package:22420/2"/>
+<part name="SV2" library="pinhead-2" deviceset="PINHD-2X12" device=""/>
 <part name="GND21" library="supply1" deviceset="GND" device=""/>
 <part name="VDD10" library="supply1" deviceset="VDD" device="" value="3V3"/>
@@
 </segment>
 </net>
-<net name="VBUS" class="0">
+<net name="N$14" class="0">
 <segment>
 <wire x1="186.69" y1="116.84" x2="184.15" y2="116.84" width="0.1524" layer="91"/>
